File: Electronics/PCB 1.0/V8_controller1.0/V8_controller1.0.kicad_pcb (KiCad board)
At the start: 2 copper layers, 95.5 x 72.7 mm, 12 parts, among them Q1 IRLZ34N, SW1 SW_SPST, U1 LM317_TO-263

Commit message: Add final gerberfiles for 1.0
Parts:
- removed R1_1: R1_1, Resistor_SMD:R_0805_2012Metric_Pad1.20x1.40mm_HandSolder
- removed R1_2: R1_2, Resistor_SMD:R_0805_2012Metric_Pad1.20x1.40mm_HandSolder
- removed U1: LM317_TO-263, Package_TO_SOT_SMD:TO-263-2
- added C2: C, Resistor_SMD:R_0805_2012Metric_Pad1.20x1.40mm_HandSolder, F.Cu at (76.3, 94.7)
- added D2: DIODE, Diode_SMD:D_SMA-SMB_Universal_Handsoldering, F.Cu at (82.7, 103.4)
- added G***: LOGO, LOGO, F.Cu at (69.5, 69.0)
- added G***: LOGO, LOGO, F.Cu at (118.0, 122.5)
- added G***: LOGO, LOGO, F.Cu at (87.0, 66.0)
- added G***: LOGO, LOGO, F.Cu at (113.5, 66.0)
- added G***: LOGO, LOGO, F.Cu at (131.0, 69.0)
- added G***: LOGO, LOGO, F.Cu at (82.0, 122.5)
- added J1: VCC 4mm banana CT3151, Connector:CalTest_CT3151, F.Cu at (128.0, 123.3)
- added J2: GND 4mm banana CT3151, Connector:CalTest_CT3151, F.Cu at (72.0, 118.2)
- added L2_1: L, Connector_JST:JST_EH_S2B-EH_1x02_P2.50mm_Horizontal, F.Cu at (72.7, 98.8)
- added L2_2: L, Connector_JST:JST_EH_S2B-EH_1x02_P2.50mm_Horizontal, F.Cu at (76.0, 107.7)
- added Q2: IRLZ34N, Package_TO_SOT_THT:TO-220-3_Horizontal_TabDown, F.Cu at (87.0, 90.5)
- added R1_3: R1_3, Resistor_SMD:R_0805_2012Metric_Pad1.20x1.40mm_HandSolder, F.Cu at (114.4, 111.5)
- added R1_VAR1: R_Variable, Resistor_THT:R_Axial_DIN0204_L3.6mm_D1.6mm_P1.90mm_Vertical, F.Cu at (114.8, 96.6)
- added R2: 100K, Resistor_SMD:R_0805_2012Metric_Pad1.20x1.40mm_HandSolder, F.Cu at (78.7, 92.4)
- added R2_SW1: 1K, Resistor_SMD:R_0805_2012Metric_Pad1.20x1.40mm_HandSolder, F.Cu at (75.0, 88.6)
- added R3_1: R1_1, Resistor_SMD:R_0805_2012Metric_Pad1.20x1.40mm_HandSolder, F.Cu at (110.5, 72.0)
- added R3_2: R3_2, Resistor_SMD:R_0805_2012Metric_Pad1.20x1.40mm_HandSolder, F.Cu at (110.5, 78.0)
- added SW2: SW_SPST, Connector_JST:JST_EH_S2B-EH_1x02_P2.50mm_Horizontal, F.Cu at (69.5, 89.9)
- added U1_2: LM338, Package_TO_SOT_THT:TO-220-3_Horizontal_TabDown, F.Cu at (97.5, 84.7)
- added U3: LM317, Package_TO_SOT_SMD:TO-263-2, F.Cu at (101.9, 119.0)
- moved D1 3.41 mm to (117.5, 103.4), turned to -111 degrees
- moved Q1 1.41 mm to (109.5, 87.0)
- moved R1 0.89 mm to (121.4, 92.3)
- moved R1_SW1 0.88 mm to (124.9, 88.8)
- moved C1 0.60 mm to (123.9, 94.9)
Connections:
- net VCC renamed Vdrive
- SW1 pad 1: Net-(R1_1-Pad2) -> VCOM
Routing:
- net GNDREF: track 0.00 -> 156.3 mm, vias 0 -> 1
- net VCOM: track 0.00 -> 139.7 mm
- net Vdrive: track 0.00 -> 133.0 mm
- net Net-(R3_1-Pad1): track 0.00 -> 125.2 mm, vias 0 -> 2
- net Net-(R1_3-Pad1): track 0.00 -> 109.5 mm, vias 0 -> 1
- net VCC: track 0.00 -> 94.2 mm
- net Net-(D2-Pad1): track 0.00 -> 40.8 mm, vias 0 -> 1
- net Net-(D1-Pad1): track 0.00 -> 39.2 mm, vias 0 -> 1
- net Net-(C1-Pad1): track 0.00 -> 24.5 mm
- net Net-(C2-Pad1): track 0.00 -> 17.8 mm
- net Net-(R2_SW1-Pad1): track 0.00 -> 5.85 mm
- net Net-(R1_SW1-Pad1): track 0.00 -> 5.70 mm
- added copper zone on B.Cu, net GNDREF
- added copper zone on F.Cu, net VCC
Other:
- board text added: "G. Abrahamsson 2022"
- board text added: "GND"
- board text added: "MAX 40VDC 5A"
- board text added: "ONLY ONE LM338 PER ENGINE"
- board text added: "V8 Solenoid engine MkI control board 1.0"
- board text added: "VCC"
